File: Board/timekillerXtreme/timekillerXtreme.kicad_pcb (KiCad board)
At the start: 2 copper layers, 61.5 x 105.2 mm, 106 parts, among them J1 Battery, J13 CONN_01X03, J15 PE7, J16 PE8, J17 PE9, J18 PE10, J19 PD4, J2 USB_OTG, J20 PD1, J21 PD0, J22 PD3, J23 PE11, J24 Pb12, J3 Conn_Bottom_Expansion, J5 Conn_LCD_Board, J6 uSD, J8 TP_AUDIO_R, J9 TP_AUDIO_L, Q1 IRLML6302, Q2 PMBT3904.215, SW1 PWR, SW2 A, SW3 B, SW4 LEFT, SW5 RIGHT, SW6 DOWN, SW7 UP, SW8 RST, U1 MCP73831, U2 FT230XS-R, U3 NCP1529, U5 STM32F407VGT6, U6 USBLC6, U7 AOZ1310, U8 USBLC6, U9 USBLC6, Y1 32.768 KHz, Y2 16MHz

Commit message: Rev. 1 updates.
Parts:
- moved D4 1.25 mm to (146.0, 46.2)
Routing:
- net (no net): track 0.00 -> 17.0 mm, vias 0 -> 1
- net GND: track 466.2 -> 463.5 mm, vias 35 -> 34
- net Net-(D4-Pad1): track 5.99 -> 4.68 mm
- net SYS_LED: track 45.1 -> 43.9 mm
- net BTN_5_A: track 125.3 -> 125.9 mm
- net AUDIO_L: track 93.9 -> 94.4 mm
Other:
- board text added: "Rev. 1 2018-10-30"
- board text removed: "Beta2 2018-10-14"
