File: Board/timekillerXtreme/timekillerXtreme.sch (KiCad schematic (older format))
At the start: 105 parts, among them J1 Battery, J10 Conn_01x02, J11 TP_USB, J12 PROG, J13 CONN_01X03, J14 TP_3.3V, J16 PE8, J17 PE9, J18 PE10, J19 PD4, J2 USB_OTG, J20 PD1, J21 PD0, J22 PD3, J23 PE11, J24 Pb12, J25 TP_BATT, J3 Conn_Bottom_Expansion, J4 Conn_Internal_Expansion, J5 Conn_LCD_Board, J6 uSD, J7 CAPTEST, J8 TP_AUDIO_R, J9 TP_AUDIO_L, Q1 IRLML6302, Q2 PMBT3904.215, SW1 PWR, SW2 A, SW3 B, SW4 LEFT, SW5 RIGHT, SW6 DOWN, SW7 UP, SW8 RST, U1 MCP73831, U2 FT230XS-R, U3 NCP1529, U4 TLV431, U5 STM32F407VGT6, U6 USBLC6, U7 AOZ1310, U8 USBLC6, U9 USBLC6, Y1 32.768 KHz, Y2 16MHz

Commit message: PCB fixes after Rev2 assembly, new assembly docs added.
Connections:
- net +3V3: now also R24.2; no longer R24.1
- net 1.2VREF: now also R24.1; no longer R24.2
Other:
- note added: "ST-Link connection:\n1 - 3.3V\n2 - SWCLK\n3 - GND\n4 - SWDIO\n5 - RST\n6 - Not connected"
- note added: "Voltage reference on pin PB1"
- note removed: "Ian is set to about 200uA"
- moved on the sheet: C1, C2, C20, C21, J12, J13, J2, J3, R24, R3, R4, SW1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
